File: pcb_activity/project/project.kicad_sch (KiCad schematic)
At the start: 13 parts, among them J1 Conn_01x08, J2 Conn_01x08

Commit message: did stuff
Parts:
- D1, D2, D3, D4, D5: footprint (none) -> LED_SMD:LED_0805_2012Metric
- J1, J2, U1: footprint (none) -> Connector_PinSocket_2.54mm:PinSocket_1x08_P2.54mm_Vertical
- R1, R2, R3, R4, R5: value R -> 1K; footprint (none) -> Resistor_SMD:R_0805_2012Metric
Connections:
- net +3.3V: now also D1.2 (A)
- net CS: now also D3.2 (A)
- net MISO: now also D5.2 (A)
- net MOSI: now also D4.2 (A)
- net SCK: now also D2.2 (A)
Other:
- moved on the sheet: D1, D2, D3, D4, D5, R1, R2, R3, R4, R5
